File: floppy featherwing rev A.brd (EAGLE design)
At the start: 50.8 x 22.9 mm, 5 parts

Commit message: floppified
Parts:
- removed JP2: (no value), pinhead:2X17
- added FDD1: FLOPPY_IDC_SHROUDED, adafruit_electromech:2X17_FLOPPY_IDC
- added R1: 2.2K, microbuilder:0805-NO
- X1: value (none) -> 3.5mm
- moved X1 0.51 mm to (9.78, 19.7)
Connections:
- removed net 3V: JP3.15, MS1.2
- new net 3.3V: JP3.15, MS1.2, R1.2
- net CHANGE: now also FDD1.34; no longer JP2.34
- net DENSITY: now also FDD1.2; no longer JP2.2
- net DIRECTION: now also FDD1.18; no longer JP2.18
- net ENABLE: now also FDD1.16; no longer JP2.16
- net GND: now also FDD1.1, FDD1.11, FDD1.13, FDD1.15, FDD1.17, FDD1.19, FDD1.21, FDD1.23, FDD1.25, FDD1.27, FDD1.29, FDD1.3, FDD1.31, FDD1.33, FDD1.5, FDD1.7, FDD1.9; no longer JP2.1, JP2.11, JP2.13, JP2.15, JP2.17, JP2.19, JP2.21, JP2.23, JP2.25, JP2.27, JP2.29, JP2.3, JP2.31, JP2.33, JP2.5, JP2.7, JP2.9
- net INDEX: now also FDD1.6; no longer JP2.8
- net PROT: now also FDD1.28; no longer JP2.28
- net READDATA: now also FDD1.30, R1.1; no longer JP2.30
- net SELECT: now also FDD1.12; no longer JP2.12
- net SIDE: now also FDD1.32; no longer JP2.32
- net STEP: now also FDD1.20; no longer JP2.20
- net TRACK0: now also FDD1.26; no longer JP2.26
- net WRITEDATA: now also FDD1.22; no longer JP2.22
- net WRITEGATE: now also FDD1.24; no longer JP2.24
Routing:
- net 3.3V: track 0.00 -> 34.5 mm, vias 0 -> 1
- net READDATA: track 11.5 -> 19.1 mm
- net 3V: track 2.54 -> 0.00 mm
- net INDEX: track 15.4 -> 17.9 mm
- net VBAT: track 3.30 -> 2.54 mm
- net USB: track 16.1 -> 16.6 mm
- net GND: track 75.6 -> 76.1 mm
Other:
- board text added: "Ch"
- board text added: "Den"
- board text added: "Dir"
- board text added: "En"
- board text added: "Idx"
- board text added: "Pr"
- board text added: "RD"
- board text added: "Sel"
- board text added: "Sid"
- board text added: "Stp"
- board text added: "Trk"
- board text added: "WD"
- board text added: "WG"
- board text removed: "1"
