File: floppy featherwing rev A.sch (EAGLE design)
At the start: 5 parts

Commit message: floppified
Parts:
- removed JP2: (no value), pinhead:PINHD-2X17
- added FDD1: FLOPPY_IDC_SHROUDED, adafruit_electromech:FLOPPY_IDC_SHROUDED
- added R1: 2.2K, microbuilder:RESISTOR0805_NOOUTLINE
- X1: value (none) -> 3.5mm
Connections:
- removed net 3V: JP3.15, MS1.3V
- new net 3.3V: JP3.15, MS1.3V, R1.2
- net CHANGE: now also FDD1.READY; no longer JP2.34
- net DENSITY: now also FDD1.DENSITY; no longer JP2.2
- net DIRECTION: now also FDD1.DIRECTION; no longer JP2.18
- net ENABLE: now also FDD1.MOTOR_ON; no longer JP2.16
- net GND: now also FDD1.GND; no longer JP2.1, JP2.11, JP2.13, JP2.15, JP2.17, JP2.19, JP2.21, JP2.23, JP2.25, JP2.27, JP2.29, JP2.3, JP2.31, JP2.33, JP2.5, JP2.7, JP2.9
- net INDEX: now also FDD1.SELECT3; no longer JP2.8
- net PROT: now also FDD1.WRITE_PROT; no longer JP2.28
- net READDATA: now also FDD1.READ_DATA, R1.1; no longer JP2.30
- net SELECT: now also FDD1.SELECT1; no longer JP2.12
- net SIDE: now also FDD1.SIDE_SELECT; no longer JP2.32
- net STEP: now also FDD1.STEP; no longer JP2.20
- net TRACK0: now also FDD1.TRACK00; no longer JP2.26
- net WRITEDATA: now also FDD1.WRITE_DATA; no longer JP2.22
- net WRITEGATE: now also FDD1.WRITE_GATE; no longer JP2.24
